Commit message: updated

File: model/robot.urdf (robot description, URDF)
Before this commit: robot unicycle, 7 links, 6 joints
Links:
- removed link body1
- removed link body2
- removed link head
- added link human, mass 50; collision box size=0.2 0.2 0.2; visual box size=0.1 0.1 0.1
- link base: mass None -> 0.001
- link left_pedal: mass None -> 0.001
- link right_pedal: mass None -> 0.001
Joints:
- removed joint body1
- removed joint body2
- removed joint head
- added joint human: type prismatic, parent base, child human, origin xyz=0 0 0 rpy=0 0 0, axis 0 1 0, limit lower=-0.1 upper=0.1 velocity=0

Commit message: updated

File: model/robot.urdf (robot description, URDF)
Before this commit: robot unicycle, 5 links, 4 joints
Links:
- link human: geometry visual box size=0.1 0.1 0.1

Commit message: updated"

File: model/robot.urdf (robot description, URDF)
Before this commit: robot unicycle, 5 links, 4 joints
Links:
- link wheel: geometry collision cylinder length=0.01 radius=0.3; visual cylinder length=0.01 radius=0.3
